File: PCB/LimitSwitch/limit_switch/limit_switch.kicad_pcb (KiCad board)
At the start: 2 copper layers, 41.5 x 22.1 mm, 15 parts, among them J1 Conn_01x03_Pin, J2 Conn_01x03_Pin, T1 Transformer_1P_1S, U1 LM358

Commit message: 5
Parts:
- removed C1: C_Small, Capacitor_SMD:C_1206_3216Metric_Pad1.33x1.80mm_HandSolder
- removed T1: Transformer_1P_1S, Transformer_THT:Transformer_Zeming_ZMPT101K
- added D1: LED, Resistor_SMD:R_0805_2012Metric_Pad1.20x1.40mm_HandSolder, F.Cu at (134.7, 105.2)
- added D4: LED, Resistor_SMD:R_0805_2012Metric_Pad1.20x1.40mm_HandSolder, F.Cu at (192.9, 139.4)
- added R10: R_Small, Resistor_SMD:R_1206_3216Metric_Pad1.30x1.75mm_HandSolder, F.Cu at (187.6, 139.7)
- added R11: R_Small, Resistor_SMD:R_1206_3216Metric_Pad1.30x1.75mm_HandSolder, F.Cu at (187.6, 143.0)
- added R12: R_Small, Resistor_SMD:R_1206_3216Metric_Pad1.30x1.75mm_HandSolder, F.Cu at (150.0, 107.5)
- added R8: R_Small, Resistor_SMD:R_1206_3216Metric_Pad1.30x1.75mm_HandSolder, F.Cu at (139.3, 103.1)
- added R9: R_Small, Resistor_SMD:R_1206_3216Metric_Pad1.30x1.75mm_HandSolder, F.Cu at (153.6, 106.2)
- added U2: PC817, Package_DIP:DIP-4_W8.89mm_SMDSocket_LongPads, F.Cu at (142.1, 107.4)
- added U3: PC817, Package_DIP:DIP-4_W8.89mm_SMDSocket_LongPads, F.Cu at (197.4, 124.8)
- added U4: PC817, Package_DIP:DIP-4_W8.89mm_SMDSocket_LongPads, F.Cu at (197.4, 131.6)
- D2, D3: value D_Small -> LED; footprint Diode_SMD:D_MicroMELF_Handsoldering -> Resistor_SMD:R_0805_2012Metric_Pad1.20x1.40mm_HandSolder
- J1: value Conn_01x03_Pin -> Conn_01x08; footprint Connector_PinHeader_2.54mm:PinHeader_1x03_P2.54mm_Vertical -> Connector_PinHeader_2.54mm:PinHeader_1x08_P2.54mm_Vertical
- J2: value Conn_01x03_Pin -> Conn_01x06; footprint Connector_PinHeader_2.54mm:PinHeader_1x03_P2.54mm_Vertical -> Connector_PinHeader_2.54mm:PinHeader_1x09_P2.54mm_Vertical
- R1: footprint Resistor_SMD:R_2512_6332Metric_Pad1.40x3.35mm_HandSolder -> Resistor_SMD:R_1206_3216Metric_Pad1.30x1.75mm_HandSolder
- R5: footprint Potentiometer_THT:Potentiometer_Bourns_3266Y_Vertical -> Resistor_SMD:R_1206_3216Metric_Pad1.30x1.75mm_HandSolder; moved to F.Cu
- U1: value LM358 -> PC817; footprint Package_SO:SO-8_3.9x4.9mm_P1.27mm -> Package_DIP:DIP-4_W8.89mm_SMDSocket_LongPads
- moved R7 68.3 mm to (187.6, 136.3), turned to 0 degrees
- moved D3 65.1 mm to (192.9, 136.4), turned to 0 degrees
- moved R3 64.6 mm to (187.6, 123.1), turned to 0 degrees
- moved R4 63.1 mm to (187.6, 126.4), turned to 0 degrees
- moved R6 60.9 mm to (187.6, 133.0), turned to 0 degrees
- moved R5 49.3 mm to (187.6, 129.7), turned to 0 degrees
- moved R2 49.2 mm to (147.7, 122.9), turned to 0 degrees
- moved J1 49.1 mm to (128.1, 124.0), turned to 180 degrees
- moved J2 47.1 mm to (158.9, 106.2)
- moved C2 36.8 mm to (167.8, 114.4), turned to 180 degrees
- moved R1 29.6 mm to (140.3, 111.8), turned to 180 degrees
- moved D2 27.9 mm to (134.7, 113.8), turned to 90 degrees
- moved U1 27.1 mm to (142.1, 116.3), turned to 0 degrees
Connections:
- D2 pad 1: Net-(D2-K) -> PIN2_IN
- D2 pad 2: GND -> Net-(D2-A)
- D3 pad 1: Net-(D3-K) -> GND
- J1 pad 1: VOUT -> GND
- J1 pad 2: VCC -> PIN4_IN
- J2 pad 1: IN2 -> VCC
- J2 pad 2: unconnected-(J2-Pin_2-Pad2) -> PIN1_OUT
- J2 pad 3: IN1 -> GND
- R1 pad 1: IN1 -> VCC
- R1 pad 2: IN2 -> Net-(D2-A)
- R2 pad 1: Net-(T1-SA) -> VCC
- R2 pad 2: IN2 -> PIN2_OUT
- R3 pad 1: Net-(D2-K) -> VCC
- R3 pad 2: Net-(T1-AB) -> PIN3_IN
- R4 pad 1: Net-(U1A-+) -> VCC
- R4 pad 2: Net-(D2-K) -> PIN3_OUT
- R5 pad 1: Net-(D3-K) -> VCC
- R5 pad 2: GND -> PIN4_IN
- R6 pad 1: GND -> VCC
- R6 pad 2: Net-(U1B--) -> PIN4_OUT
- R7 pad 1: Net-(U1B--) -> PIN2_OUT
- R7 pad 2: VOUT -> GND
- U1 pad 1: Net-(D3-A) -> PIN2_IN
- U1 pad 2: Net-(D3-K) -> GND
- U1 pad 3: Net-(U1A-+) -> GND
- U1 pad 4: GND -> PIN2_OUT
Routing:
- net Net-(D3-K): track 18.1 -> 0.00 mm
- net VOUT: track 17.1 -> 0.00 mm
- net Net-(U1A-+): track 16.1 -> 0.00 mm
- net GND: track 54.6 -> 67.5 mm
- net PIN2_OUT: track 0.00 -> 12.8 mm
- net PIN2_IN: track 0.00 -> 11.1 mm
- net IN1: track 10.1 -> 0.00 mm
- net PIN1_IN: track 0.00 -> 9.53 mm
- net IN2: track 7.95 -> 0.00 mm
- net VCC: track 21.2 -> 28.8 mm, vias 2 -> 0
- net Net-(U1B--): track 7.06 -> 0.00 mm
- net PIN1_OUT: track 0.00 -> 6.02 mm
- net Net-(D2-K): track 5.93 -> 0.00 mm
- net Net-(D2-A): track 0.00 -> 4.43 mm
- net Net-(T1-SA): track 3.72 -> 0.00 mm
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Other:
- board outline removed
- board text removed: "${REFERENCE}"
