File: PCB/LimitSwitch/limit_switch/limit_switch-rounded.kicad_pcb (KiCad board)
At the start: 2 copper layers, 40.6 x 38.1 mm, 30 parts, among them J2 Conn_01x06, J3 Conn_01x08, J4 Conn_01x08, J5 Conn_01x08, J6 Conn_01x08, U1 PC817, U2 PC817, U3 PC817, U4 PC817

Commit message: 4
Routing:
- net GND: track 158.9 -> 157.1 mm
- net VCC: track 62.3 -> 63.0 mm

Commit message: 3
Routing:
- net PIN1_OUT: track 0.00 -> 9.05 mm
- net GND: vias 0 -> 3
- net (no net): vias 4 -> 0
Other:
- board size 40.6 x 38.1 mm -> 42.2 x 39.6 mm
