File: ExternalBoard/PCB/ExternalBoard/ExternalBoard.kicad_pcb (KiCad board)
At the start: 2 copper layers, 2 parts, among them U1 REF01CP

Commit message: 3
Parts:
- added C1: C_Small, Capacitor_SMD:C_1206_3216Metric, F.Cu at (208.3, 139.1)
- added C2: C_Small, Capacitor_SMD:C_1206_3216Metric, F.Cu at (221.0, 138.2)
- added D5: ~, ESP32_S2:StepDown, F.Cu at (171.2, 113.4)
- added D6: D_Small, Diode_SMD:D_SMA, F.Cu at (169.1, 138.2)
- added D7: D_Small, Diode_SMD:D_SMF, F.Cu at (202.2, 106.8)
- added J1: Conn_01x04_Pin, Connector_PinHeader_2.54mm:PinHeader_1x04_P2.54mm_Vertical, F.Cu at (173.2, 127.0)
- added J10: Conn_01x04_Pin, ESP32_S2:PIN0, F.Cu at (214.9, 121.9)
- added J11: Conn_01x04_Pin, ESP32_S2:PIN0, F.Cu at (214.9, 119.4)
- added J12: Conn_01x04_Pin, ESP32_S2:PIN0, F.Cu at (214.9, 116.8)
- added J13: Conn_01x04_Pin, Connector_PinHeader_2.54mm:PinHeader_1x02_P2.54mm_Vertical, F.Cu at (226.1, 108.2)
- added J14: Conn_01x04_Pin, ESP32_S2:PIN0, F.Cu at (218.9, 116.8)
- added J15: Conn_01x04_Pin, ESP32_S2:PIN0, F.Cu at (218.9, 119.4)
- added J16: Conn_01x04_Pin, ESP32_S2:PIN0, F.Cu at (218.9, 121.9)
- added J17: Conn_01x04_Pin, ESP32_S2:PIN0, F.Cu at (218.9, 124.5)
- added J18: Conn_01x04_Pin, ESP32_S2:PIN0, F.Cu at (218.9, 127.0)
- added J19: Conn_01x04_Pin, ESP32_S2:PIN0, F.Cu at (218.9, 129.5)
- added J2: Conn_01x04_Pin, Connector_PinHeader_2.54mm:PinHeader_1x02_P2.54mm_Vertical, F.Cu at (167.7, 97.5)
- added J20: Conn_01x04_Pin, ESP32_S2:PIN0, F.Cu at (218.9, 132.1)
- added J21: Conn_01x04_Pin, ESP32_S2:PIN0, F.Cu at (227.1, 116.9)
- added J22: Conn_01x04_Pin, ESP32_S2:PIN0, F.Cu at (227.1, 119.4)
- added J23: Conn_01x04_Pin, ESP32_S2:PIN0, F.Cu at (227.1, 121.9)
- added J24: Conn_01x04_Pin, ESP32_S2:PIN0, F.Cu at (227.1, 124.5)
- added J25: Conn_01x04_Pin, ESP32_S2:PIN0, F.Cu at (227.1, 127.0)
- added J26: Conn_01x04_Pin, ESP32_S2:PIN0, F.Cu at (227.1, 129.6)
- added J27: Conn_01x04_Pin, ESP32_S2:PIN0, F.Cu at (227.1, 132.1)
- added J28: Conn_01x04_Pin, ESP32_S2:PIN0, F.Cu at (223.0, 116.8)
- added J29: Conn_01x04_Pin, ESP32_S2:PIN0, F.Cu at (223.0, 119.4)
- added J3: Conn_01x04_Pin, ESP32_S2:PIN0, F.Cu at (210.8, 119.4)
- added J30: Conn_01x04_Pin, ESP32_S2:PIN0, F.Cu at (223.0, 121.9)
- added J31: Conn_01x04_Pin, ESP32_S2:PIN0, F.Cu at (223.0, 124.5)
- added J32: Conn_01x04_Pin, ESP32_S2:PIN0, F.Cu at (223.0, 127.0)
- added J33: Conn_01x04_Pin, ESP32_S2:PIN0, F.Cu at (223.0, 129.5)
- added J34: Conn_01x04_Pin, ESP32_S2:PIN0, F.Cu at (223.0, 132.1)
- added J4: Conn_01x04_Pin, ESP32_S2:PIN0, F.Cu at (210.8, 121.9)
- added J5: Conn_01x04_Pin, ESP32_S2:PIN0, F.Cu at (210.8, 124.5)
- added J6: Conn_01x04_Pin, ESP32_S2:PIN0, F.Cu at (210.8, 127.0)
- added J7: Conn_01x04_Pin, ESP32_S2:PIN0, F.Cu at (214.9, 129.5)
- added J8: Conn_01x04_Pin, ESP32_S2:PIN0, F.Cu at (214.9, 127.0)
- added J9: Conn_01x04_Pin, ESP32_S2:PIN0, F.Cu at (214.9, 124.5)
- added Q3: IRFS4229, Package_TO_SOT_SMD:TO-263-2, F.Cu at (217.1, 108.0)
- added R4: R_Small, Resistor_SMD:R_1206_3216Metric_Pad1.30x1.75mm_HandSolder, F.Cu at (205.2, 106.7)
- added R5: R_Small, Resistor_SMD:R_1206_3216Metric_Pad1.30x1.75mm_HandSolder, F.Cu at (189.5, 101.6)
- added R6: R_Small, Resistor_SMD:R_1206_3216Metric_Pad1.30x1.75mm_HandSolder, F.Cu at (191.0, 117.9)
- added U3: AMS1117-3.3, Package_TO_SOT_SMD:SOT-223-3_TabPin2, F.Cu at (215.0, 139.7)
- D1: footprint ESP32_S2:ESP32_S2 -> ESP32_S2:ESP32_S2_V2
- U1: value REF01CP -> PC817; footprint Package_DIP:DIP-8_W7.62mm -> Package_DIP:DIP-4_W7.62mm
- moved D1 101.7 mm to (194.7, 124.5)
- moved U1 95.7 mm to (194.6, 109.7), turned to 90 degrees
Connections:
- D1 pad 16: unconnected-(D1-Pad16) -> /TX
- D1 pad 18: unconnected-(D1-Pad18) -> /RX
- D1 pad 39: Net-(U1-VIN) -> unconnected-(D1-Pad39)
- D1 pad GND: unconnected-(D1-PadGND) -> /GND
- D1 pad VBUS: Net-(U1-GND) -> /V5
- U1 pad 1: unconnected-(U1-NC-Pad1) -> Net-(R6-Pad1)
- U1 pad 2: Net-(U1-VIN) -> /GND
- U1 pad 3: unconnected-(U1-TEMP-Pad3) -> Net-(D7-K)
- U1 pad 4: Net-(U1-GND) -> Net-(R5-Pad1)
Routing:
- net /GND: track 0.00 -> 139.2 mm
- net /V5: track 0.00 -> 87.8 mm
- net Net-(J28-Pin_1): track 0.00 -> 33.7 mm
- net Net-(J9-Pin_1): track 0.00 -> 20.8 mm, vias 0 -> 2
- net Net-(J8-Pin_1): track 0.00 -> 20.8 mm, vias 0 -> 2
- net Net-(J7-Pin_1): track 0.00 -> 20.8 mm, vias 0 -> 2
- net Net-(J12-Pin_1): track 0.00 -> 20.8 mm, vias 0 -> 2
- net Net-(J11-Pin_1): track 0.00 -> 20.8 mm, vias 0 -> 2
- net Net-(J10-Pin_1): track 0.00 -> 20.8 mm, vias 0 -> 2
- net Net-(D6-A): track 0.00 -> 16.9 mm
- net Net-(D7-K): track 0.00 -> 13.8 mm
- net Net-(R6-Pad1): track 0.00 -> 9.37 mm
- net /TX: track 0.00 -> 7.44 mm
- net /RX: track 0.00 -> 7.44 mm
- net /V_IN: track 0.00 -> 5.39 mm
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